File: Front_Panel/Front_Panel.kicad_pcb (KiCad board)
At the start: 2 copper layers, 160 x 70 mm, 27 parts, among them J2 Conn_01x05, Q1 BC817, SW1 SW_Push, SW2 SW_Push, SW3 SW_Push, SW4 SW_Push, U1 NHD-C0220BIZ, U2 MCP23008-xSO

Commit message: added PCB layou
Routing:
- net +3.3V: track 265.8 -> 264.4 mm
Other:
- outline, holes or cut-outs redrawn
Changed lines of the file:
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@@
 		(tags "mountinghole M4 DIN965")
 		(property "Reference" "H2"
-			(at 0 -4.7 0)
+			(at 0 -5 0)
 			(layer "F.SilkS")
 			(effects
@@
 		(tags "mountinghole M4 DIN965")
 		(property "Reference" "H1"
-			(at 0 -4.7 0)
+			(at 0 5 0)
 			(layer "F.SilkS")
 			(effects
@@
 		(tags "mountinghole M4 DIN965")
 		(property "Reference" "H3"
-			(at 0 -4.7 0)
+			(at 0 5 0)
 			(layer "F.SilkS")
 			(effects
@@
 		(tags "mountinghole M4 DIN965")
 		(property "Reference" "H4"
-			(at 0 -4.7 0)
+			(at 0 -5 0)
 			(layer "F.SilkS")
 			(effects
@@
 	)
 	(gr_line
-		(start 73 72.5)
-		(end 223 72.5)
+		(start 223.7 142.5)
+		(end 72.3 142.5)
 		(stroke
 			(width 0.05)
@@
 	)
 	(gr_line
-		(start 68 137.5)
-		(end 68 77.5)
+		(start 72.3 72.5)
+		(end 223.7 72.5)
 		(stroke
 			(width 0.05)
@@
 	)
 	(gr_arc
-		(start 68 77.5)
-		(mid 69.464466 73.964466)
-		(end 73 72.5)
+		(start 72.3 142.5)
+		(mid 69.259441 141.240559)
+		(end 68 138.2)
 		(stroke
 			(width 0.05)
@@
 		(layer "Edge.Cuts")
 	)
-	(gr_line
-		(start 223 142.5)
-		(end 73 142.5)
+	(gr_arc
+		(start 223.7 72.5)
+		(mid 226.740559 73.759441)
+		(end 228 76.8)
 		(stroke
 			(width 0.05)
@@
 	)
 	(gr_line
-		(start 228 77.5)
-		(end 228 137.5)
+		(start 228 76.8)
+		(end 228 138.2)
 		(stroke
 			(width 0.05)
@@
 	)
 	(gr_arc
-		(start 223 72.5)
-		(mid 226.535534 73.964466)
-		(end 228 77.5)
+		(start 68 76.8)
+		(mid 69.259441 73.759441)
+		(end 72.3 72.5)
 		(stroke
 			(width 0.05)
@@
 	)
 	(gr_arc
-		(start 228 137.5)
-		(mid 226.535534 141.035534)
-		(end 223 142.5)
+		(start 228 138.2)
+		(mid 226.740559 141.240559)
+		(end 223.7 142.5)
 		(stroke
 			(width 0.05)
@@
 		(layer "Edge.Cuts")
 	)
-	(gr_arc
-		(start 73 142.5)
-		(mid 69.464466 141.035534)
-		(end 68 137.5)
+	(gr_line
+		(start 68 138.2)
+		(end 68 76.8)
 		(stroke
 			(width 0.05)
@@
 	)
 	(segment
+		(start 151.54 136.46)
+		(end 151.54 125.96)
+		(width 0.75)
+		(layer "F.Cu")
+		(net 1)
+	)
+	(segment
 		(start 177 116.05)
 		(end 173.2875 116.05)
@@
 	)
 	(segment
-		(start 151 126.5)
-		(end 151.54 125.96)
-		(width 0.75)
-		(layer "F.Cu")
-		(net 1)
-	)
-	(segment
-		(start 127.5 128.25)
-		(end 127.25 128.5)
-		(width 0.75)
-		(layer "F.Cu")
-		(net 1)
-	)
-	(segment
 		(start 151.54 125.96)
 		(end 154.08 123.42)
@@
 	)
 	(segment
-		(start 126.5 128.25)
-		(end 127.5 127.25)
+		(start 114.8 119.55)
+		(end 114.8 112.25)
 		(width 0.75)
 		(layer "F.Cu")
@@
 	)
 	(segment
-		(start 114.8 119.55)
-		(end 114.8 112.25)
+		(start 120.125 123.125)
+		(end 124.25 127.25)
 		(width 0.75)
 		(layer "F.Cu")
@@
 	)
 	(segment
-		(start 150.5 137.5)
-		(end 151.54 136.46)
+		(start 148.6 125.96)
+		(end 148.6 127.23)
 		(width 0.75)
 		(layer "F.Cu")
@@
 	)
 	(segment
-		(start 151.54 136.46)
-		(end 151.54 125.96)
-		(width 0.75)
-		(layer "F.Cu")
-		(net 1)
-	)
-	(segment
 		(start 120.125 123.125)
 		(end 116.55 119.55)
@@
 	)
 	(segment
-		(start 148.6 126.4)
-		(end 148.6 125.96)
-		(width 0.75)
-		(layer "F.Cu")
-		(net 1)
-	)
-	(segment
-		(start 127.25 128.5)
-		(end 127.25 136.5)
-		(width 0.75)
-		(layer "F.Cu")
-		(net 1)
-	)
-	(segment
-		(start 148.5 126.5)
-		(end 148.6 126.4)
-		(width 0.75)
-		(layer "F.Cu")
-		(net 1)
-	)
-	(segment
 		(start 177 122.75)
 		(end 178 123.75)
@@
 	)
 	(segment
-		(start 148.5 126.5)
-		(end 151 126.5)
+		(start 127.5 136.75)
+		(end 128.25 137.5)
 		(width 0.75)
 		(layer "F.Cu")
@@
 	)
 	(segment
-		(start 157.93 123.45)
-		(end 157.9 123.42)
+		(start 150.5 137.5)
+		(end 151.54 136.46)
 		(width 0.75)
 		(layer "F.Cu")
@@
 	)
 	(segment
-		(start 148.5 126.5)
-		(end 148.6 126.6)
+		(start 157.93 123.45)
+		(end 157.9 123.42)
 		(width 0.75)
 		(layer "F.Cu")
@@
 	)
 	(segment
-		(start 127.5 127.25)
-		(end 127.5 128.25)
+		(start 124.25 127.25)
+		(end 127.5 127.25)
 		(width 0.75)
 		(layer "F.Cu")
@@
 	)
 	(segment
-		(start 120.125 123.125)
-		(end 125.25 128.25)
+		(start 151.54 125.96)
+		(end 148.6 125.96)
 		(width 0.75)
 		(layer "F.Cu")
@@
 	)
 	(segment
-		(start 160.75 123.45)
-		(end 157.93 123.45)
+		(start 127.5 127.25)
+		(end 127.5 136.75)
 		(width 0.75)
 		(layer "F.Cu")
@@
 	)
 	(segment
-		(start 148.6 126.6)
-		(end 148.6 127.23)
+		(start 160.75 123.45)
+		(end 157.93 123.45)
 		(width 0.75)
 		(layer "F.Cu")
@@
 	)
 	(segment
-		(start 119.25 124)
-		(end 120.125 123.125)
+		(start 128.25 137.5)
+		(end 150.5 137.5)
 		(width 0.75)
 		(layer "F.Cu")
@@
 	)
 	(segment
-		(start 128.25 137.5)
-		(end 150.5 137.5)
+		(start 119.25 124)
+		(end 120.125 123.125)
 		(width 0.75)
 		(layer "F.Cu")
@@
 	)
 	(segment
-		(start 127.25 136.5)
-		(end 128.25 137.5)
-		(width 0.75)
-		(layer "F.Cu")
-		(net 1)
-	)
-	(segment
-		(start 125.25 128.25)
-		(end 126.5 128.25)
-		(width 0.75)
-		(layer "F.Cu")
-		(net 1)
-	)
-	(segment
 		(start 178 123.75)
 		(end 178.0875 123.75)
@@
 		(polygon
 			(pts
-				(xy 66 146) (xy 66.5 146.5) (xy 232.5 146.5) (xy 232.5 69.75) (xy 231.75 69) (xy 66 69) (xy 66 72.5)
+				(xy 66 146.5) (xy 232.5 146.5) (xy 232.5 69) (xy 66 69)
 			)
 		)
@@
 		(polygon
 			(pts
-				(xy 66 69) (xy 66 146) (xy 66.5 146.5) (xy 232.5 146.5) (xy 232.5 69.75) (xy 231.75 69)
+				(xy 66 69) (xy 66 146.5) (xy 232.5 146.5) (xy 232.5 69)
 			)
 		)
